Commit message: turned all components into macros

File: urdf/olv-cam01.urdf (robot description, URDF)
Before this commit: robot olv-cam01, 1 links, 0 joints
Links:
- link base_link: geometry 

File: urdf/olv-srv01.urdf (robot description, URDF)
Before this commit: robot olv-srv01, 1 links, 0 joints
Links:
- link base_link: geometry 
