Commit message: Renamed package

File: urdf/olv-cam01.urdf.xacro (robot description, xacro)
@@ -15,5 +15,5 @@
       <visual>
         <geometry>
-          <mesh filename="package://olive_components_description/meshes/olv-cam01.dae" />
+          <mesh filename="package://olive_modules_description/meshes/olv-cam01.dae" />
         </geometry>
       </visual>

File: urdf/olv-imu01.urdf (robot description, URDF)
Before this commit: robot olv-imu01, 1 links, 0 joints
Links:
- link base_link: geometry collision box size=0.04 0.04 0.018; visual mesh filename=package://olive_modules_description/meshes/olv-imu01.dae

File: urdf/olv-srv01.urdf.xacro (robot description, xacro)
@@ -14,5 +14,5 @@
       <visual>
         <geometry>
-          <mesh filename="package://olive_components_description/meshes/olv-srv01-body.dae" />
+          <mesh filename="package://olive_modules_description/meshes/olv-srv01-body.dae" />
         </geometry>
       </visual>
@@ -26,5 +26,5 @@
       <visual>
         <geometry>
-          <mesh filename="package://olive_components_description/meshes/olv-srv01-horn.dae" />
+          <mesh filename="package://olive_modules_description/meshes/olv-srv01-horn.dae" />
         </geometry>
         <material name="blue">

Commit message: Added side links to each module

File: urdf/olv-cam01.urdf.xacro (robot description, xacro)
@@ -20,35 +20,68 @@
       <collision>
         <geometry>
-          <box size="0.04 0.04 0.046" />
+          <box size="0.04 0.04 0.04" />
         </geometry>
+        <origin xyz="0 0 0.005" />
       </collision>
     </link>
+    <link name="${namespace}_bottom_link" />
+    <link name="${namespace}_right_link" />
+    <link name="${namespace}_left_link"/>
+    <link name="${namespace}_back_link"/>
+    <link name="${namespace}_camera_link"/>
     <!-- Check for unexpected value and print warning -->
-    <xacro:if value="${mounting_side != 'bottom' and mounting_side != 'back' and mounting_side != 'left' and mounting_side != 'right'}">
-        <xacro:warning>Unexpected value for mounting_side in olv-cam01 macro. Accepted values are 'bottom', 'back', 'left', 'right'. Using default 'bottom'.</xacro:warning>
-        <xacro:property name="mounting_side" value="bottom"/>
+    <xacro:if
+      value="${mounting_side != 'bottom' and mounting_side != 'back' and mounting_side != 'left' and mounting_side != 'right'}">
+      <xacro:warning>Unexpected value for mounting_side in olv-cam01 macro. Accepted values are
+        'bottom', 'back', 'left', 'right'. Using default 'bottom'.</xacro:warning>
+      <xacro:property name="mounting_side" value="bottom" />
     </xacro:if>
     <!-- Conditional translations based on mount_frame -->
     <xacro:if value="${mounting_side == 'bottom'}">
-        <xacro:property name="mount_translation" value="0 0 0.015"/>
-        <xacro:property name="mount_rotation" value="0 0 ${mounting_rotation}"/>
+      <xacro:property name="mount_translation" value="0 0 0.015" />
+      <xacro:property name="mount_rotation" value="0 0 ${mounting_rotation}" />
     </xacro:if>
     <xacro:if value="${mounting_side == 'back'}">
-      <xacro:property name="mount_translation" value="0 0 0.02"/>
-      <xacro:property name="mount_rotation" value="0 -1.5707963267948966 ${mounting_rotation}"/>
+      <xacro:property name="mount_translation" value="0 0 0.02" />
+      <xacro:property name="mount_rotation" value="0 -1.57079632679 ${mounting_rotation}" />
     </xacro:if>
     <xacro:if value="${mounting_side == 'left'}">
-      <xacro:property name="mount_translation" value="0 0 0.02"/>
-      <xacro:property name="mount_rotation" value="1.5707963267948966 0 ${mounting_rotation}"/>
+      <xacro:property name="mount_translation" value="0 0 0.02" />
+      <xacro:property name="mount_rotation" value="1.57079632679 0 ${mounting_rotation}" />
     </xacro:if>
     <xacro:if value="${mounting_side == 'right'}">
-      <xacro:property name="mount_translation" value="0 0 0.02"/>
-      <xacro:property name="mount_rotation" value="-1.5707963267948966 0 ${mounting_rotation}"/>
+      <xacro:property name="mount_translation" value="0 0 0.02" />
+      <xacro:property name="mount_rotation" value="-1.57079632679 0 ${mounting_rotation}" />
     </xacro:if>
-    <joint name="${namespace}_base_joint" type="fixed">
+    <joint name="${namespace}_body_joint" type="fixed">
       <parent link="${parent_link}" />
       <child link="${namespace}_body_link" />
       <origin xyz="${mount_translation}" rpy="${mount_rotation}" />
     </joint>
+    <joint name="${namespace}_bottom_joint" type="fixed">
+      <parent link="${namespace}_body_link" />
+      <child link="${namespace}_bottom_link" />
+      <origin xyz="0 0 -0.015" rpy="3.14159265359 0 -1.57079632679" />
+    </joint>
+    <joint name="${namespace}_right_joint" type="fixed">
+      <parent link="${namespace}_body_link" />
+      <child link="${namespace}_right_link" />
+      <origin xyz="0 0.02 0" rpy="-1.57079632679 3.14159265359 0" />
+    </joint>
+    <joint name="${namespace}_left_joint" type="fixed">
+      <parent link="${namespace}_body_link" />
+      <child link="${namespace}_left_link" />
+      <origin xyz="0 -0.02 0" rpy="1.57079632679 0 0" />
+    </joint>
+    <joint name="${namespace}_back_joint" type="fixed">
+      <parent link="${namespace}_body_link" />
+      <child link="${namespace}_back_link" />
+      <origin xyz="-0.02 0 0" rpy="1.57079632679 0 -1.57079632679" />
+    </joint>
+    <joint name="${namespace}_camera_joint" type="fixed">
+      <parent link="${namespace}_body_link" />
+      <child link="${namespace}_camera_link" />
+      <origin xyz="0 0 0.02" rpy="0 0 0" />
+    </joint>
   </xacro:macro>
 </robot>

File: urdf/olv-imu01.urdf (robot description, URDF)
Before this commit: robot olv-imu01, 1 links, 0 joints
Links:
- link base_link: geometry 

File: urdf/olv-srv01.urdf.xacro (robot description, xacro)
@@ -28,9 +28,10 @@
           <mesh filename="package://olive_modules_description/meshes/olv-srv01-horn.dae" />
         </geometry>
-        <material name="blue">
-          <color rgba="0 0 1 1" /> <!-- RGBA for blue color -->
-        </material>
       </visual>
     </link>
+    <link name="${namespace}_bottom_link" />
+    <link name="${namespace}_right_link" />
+    <link name="${namespace}_left_link"/>
+    <link name="${namespace}_back_link"/>
     <!-- Check for unexpected value and print warning -->
     <xacro:if value="${mounting_side != 'bottom' and mounting_side != 'back' and mounting_side != 'left' and mounting_side != 'right'}">
@@ -45,13 +46,13 @@
     <xacro:if value="${mounting_side == 'back'}">
       <xacro:property name="mount_translation" value="0 0 0.03"/>
-      <xacro:property name="mount_rotation" value="0 -1.5707963267948966 ${mounting_rotation}"/>
+      <xacro:property name="mount_rotation" value="0 -1.57079632679 ${mounting_rotation}"/>
     </xacro:if>
     <xacro:if value="${mounting_side == 'left'}">
       <xacro:property name="mount_translation" value="0 0 0.03"/>
-      <xacro:property name="mount_rotation" value="1.5707963267948966 0 ${mounting_rotation}"/>
+      <xacro:property name="mount_rotation" value="1.57079632679 0 ${mounting_rotation}"/>
     </xacro:if>
     <xacro:if value="${mounting_side == 'right'}">
       <xacro:property name="mount_translation" value="0 0 0.03"/>
-      <xacro:property name="mount_rotation" value="-1.5707963267948966 0 ${mounting_rotation}"/>
+      <xacro:property name="mount_rotation" value="-1.57079632679 0 ${mounting_rotation}"/>
     </xacro:if>
     <joint name="${namespace}_base_joint" type="fixed">
@@ -66,4 +67,24 @@
       <axis xyz="0 0 1" />
     </joint>
+    <joint name="${namespace}_bottom_joint" type="fixed">
+      <parent link="${namespace}_body_link" />
+      <child link="${namespace}_bottom_link" />
+      <origin xyz="0 0 -0.023" rpy="3.14159265359 0 -1.57079632679" />
+    </joint>
+    <joint name="${namespace}_right_joint" type="fixed">
+      <parent link="${namespace}_body_link" />
+      <child link="${namespace}_right_link" />
+      <origin xyz="0 0.03 0" rpy="-1.57079632679 3.14159265359 0" />
+    </joint>
+    <joint name="${namespace}_left_joint" type="fixed">
+      <parent link="${namespace}_body_link" />
+      <child link="${namespace}_left_link" />
+      <origin xyz="0 -0.03 0" rpy="1.57079632679 0 0" />
+    </joint>
+    <joint name="${namespace}_back_joint" type="fixed">
+      <parent link="${namespace}_body_link" />
+      <child link="${namespace}_back_link" />
+      <origin xyz="-0.03 0 0" rpy="1.57079632679 0 -1.57079632679" />
+    </joint>
   </xacro:macro>
 </robot>

Commit message: Changed package name

File: urdf/olv-cam01.urdf.xacro (robot description, xacro)
@@ -15,5 +15,5 @@
       <visual>
         <geometry>
-          <mesh filename="package://olive_modules_description/meshes/olv-cam01.dae" />
+          <mesh filename="package://olv_module_descriptions/meshes/olv-cam01.dae" />
         </geometry>
       </visual>

File: urdf/olv-imu01.urdf.xacro (robot description, xacro)
@@ -15,5 +15,5 @@
       <visual>
         <geometry>
-          <mesh filename="package://olive_modules_description/meshes/olv-imu01.dae" />
+          <mesh filename="package://olv_module_descriptions/meshes/olv-imu01.dae" />
         </geometry>
       </visual>

File: urdf/olv-srv01.urdf.xacro (robot description, xacro)
@@ -14,5 +14,5 @@
       <visual>
         <geometry>
-          <mesh filename="package://olive_modules_description/meshes/olv-srv01-body.dae" />
+          <mesh filename="package://olv_module_descriptions/meshes/olv-srv01-body.dae" />
         </geometry>
       </visual>
@@ -26,5 +26,5 @@
       <visual>
         <geometry>
-          <mesh filename="package://olive_modules_description/meshes/olv-srv01-horn.dae" />
+          <mesh filename="package://olv_module_descriptions/meshes/olv-srv01-horn.dae" />
         </geometry>
       </visual>
