Commit message: removed top links from gns and rad

File: urdf/olv-gnx01.urdf.xacro (robot description, xacro)
@@ -20,13 +20,13 @@
       <collision>
         <geometry>
-          <box size="0.04 0.04 0.018" />
+          <box size="0.04 0.04 0.032"/>
         </geometry>
+        <origin xyz="0 0 0.008" />
       </collision>
     </link>
     <link name="${namespace}_bottom_link" />
-    <link name="${namespace}_top_link"/>
     <!-- Check for unexpected value and print warning -->
     <xacro:if
-      value="${mounting_side != 'bottom' and mounting_side != 'top'}">
+      value="${mounting_side != 'bottom'}">
       <xacro:warning>Unexpected value for mounting_side in olv-gnx01 macro. Accepted values are
         'bottom', 'top'. Using default 'bottom'.</xacro:warning>
@@ -37,8 +37,4 @@
       <xacro:property name="mount_translation" value="0 0 0.009" />
       <xacro:property name="mount_rotation" value="0 0 ${mounting_rotation}" />
-    </xacro:if>
-    <xacro:if value="${mounting_side == 'top'}">
-      <xacro:property name="mount_translation" value="0 0 0.009" />
-      <xacro:property name="mount_rotation" value="0 3.14159265359 ${mounting_rotation}" />
     </xacro:if>
     <joint name="${namespace}_body_joint" type="fixed">
@@ -52,9 +48,4 @@
       <origin xyz="0 0 -0.009" rpy="3.14159265359 0 -1.57079632679" />
     </joint>
-    <joint name="${namespace}_right_joint" type="fixed">
-      <parent link="${namespace}_body_link" />
-      <child link="${namespace}_top_link" />
-      <origin xyz="0 0 0.009" rpy="0 0 0" />
-    </joint>
   </xacro:macro>
 </robot>

File: urdf/olv-n5g01.urdf.xacro (robot description, xacro)
@@ -7,5 +7,5 @@
     - parent_link: Define which link the n5g is mounted to
     - mounting_side: Specifies the mounting side of the cam.
-      Acceptable values are: 'bottom', 'top'
+      Acceptable values are: 'lower', 'right'
     - mounting_rotation: Specifies an additional rotation around the n5g's mounting frame's z-axis
 -->
@@ -24,19 +24,19 @@
       </collision>
     </link>
-    <link name="${namespace}_bottom_link" />
-    <link name="${namespace}_top_link"/>
+    <link name="${namespace}_right_link" />
+    <link name="${namespace}_lower_link"/>
     <!-- Check for unexpected value and print warning -->
     <xacro:if
-      value="${mounting_side != 'bottom' and mounting_side != 'top'}">
+      value="${mounting_side != 'right' and mounting_side != 'lower'}">
       <xacro:warning>Unexpected value for mounting_side in olv-n5g01 macro. Accepted values are
-        'bottom', 'top'. Using default 'bottom'.</xacro:warning>
-      <xacro:property name="mounting_side" value="bottom" />
+        'right', 'lower'. Using default 'right'.</xacro:warning>
+      <xacro:property name="mounting_side" value="right" />
     </xacro:if>
     <!-- Conditional translations based on mount_frame -->
-    <xacro:if value="${mounting_side == 'bottom'}">
+    <xacro:if value="${mounting_side == 'right'}">
       <xacro:property name="mount_translation" value="0 0 0.009" />
       <xacro:property name="mount_rotation" value="0 0 ${mounting_rotation}" />
     </xacro:if>
-    <xacro:if value="${mounting_side == 'top'}">
+    <xacro:if value="${mounting_side == 'lower'}">
       <xacro:property name="mount_translation" value="0 0 0.009" />
       <xacro:property name="mount_rotation" value="0 3.14159265359 ${mounting_rotation}" />
@@ -47,12 +47,12 @@
       <origin xyz="${mount_translation}" rpy="${mount_rotation}" />
     </joint>
-    <joint name="${namespace}_bottom_joint" type="fixed">
+    <joint name="${namespace}_right_joint" type="fixed">
       <parent link="${namespace}_body_link" />
-      <child link="${namespace}_bottom_link" />
+      <child link="${namespace}_right_link" />
       <origin xyz="0 0 -0.009" rpy="3.14159265359 0 -1.57079632679" />
     </joint>
-    <joint name="${namespace}_right_joint" type="fixed">
+    <joint name="${namespace}_lower_joint" type="fixed">
       <parent link="${namespace}_body_link" />
-      <child link="${namespace}_top_link" />
+      <child link="${namespace}_lower_link" />
       <origin xyz="0 0 0.009" rpy="0 0 0" />
     </joint>

File: urdf/olv-rad01.urdf.xacro (robot description, xacro)
@@ -20,13 +20,13 @@
       <collision>
         <geometry>
-          <box size="0.04 0.04 0.018" />
+          <box size="0.04 0.04 0.032"/>
         </geometry>
+        <origin xyz="0 0 0.008" />
       </collision>
     </link>
     <link name="${namespace}_bottom_link" />
-    <link name="${namespace}_top_link"/>
     <!-- Check for unexpected value and print warning -->
     <xacro:if
-      value="${mounting_side != 'bottom' and mounting_side != 'top'}">
+      value="${mounting_side != 'bottom'}">
       <xacro:warning>Unexpected value for mounting_side in olv-rad01 macro. Accepted values are
         'bottom', 'top'. Using default 'bottom'.</xacro:warning>
@@ -37,8 +37,4 @@
       <xacro:property name="mount_translation" value="0 0 0.009" />
       <xacro:property name="mount_rotation" value="0 0 ${mounting_rotation}" />
-    </xacro:if>
-    <xacro:if value="${mounting_side == 'top'}">
-      <xacro:property name="mount_translation" value="0 0 0.009" />
-      <xacro:property name="mount_rotation" value="0 3.14159265359 ${mounting_rotation}" />
     </xacro:if>
     <joint name="${namespace}_body_joint" type="fixed">
@@ -52,9 +48,4 @@
       <origin xyz="0 0 -0.009" rpy="3.14159265359 0 -1.57079632679" />
     </joint>
-    <joint name="${namespace}_right_joint" type="fixed">
-      <parent link="${namespace}_body_link" />
-      <child link="${namespace}_top_link" />
-      <origin xyz="0 0 0.009" rpy="0 0 0" />
-    </joint>
   </xacro:macro>
 </robot>
